File: synth/SWEEP_VFO.sch (KiCad schematic (older format))
At the start: 19 parts

Commit message: automated commit
Parts:
- removed Q?: Q_PNP_EBC, symbol Device:Q_PNP_EBC
- removed R? (x3): 10k, symbol Device:R
- removed R?: 30k, symbol Device:R
- removed R?: 330, symbol Device:R
- removed RV?: 10k, symbol Device:R_POT
- removed U? (x5): LMC660, Package_DIP:DIP-14_W7.62mm_LongPads, symbol custom:LMC660
- removed U?: R20407RN02Q, symbol custom:R20407RN02Q
- added Q?: BC549BTA, symbol Device:Q_NPN_CBE
- added Q?: BC556BTA, symbol Device:Q_PNP_CBE
- added R? (x3): 10k, symbol Device:R
- added R? (x2): 3k3, symbol Device:R
- added RV? (x4): 10k, symbol Device:R_POT
- added SW?: SW_SPDT, symbol Switch:SW_SPDT
- added U? (x5): MCP6004, Package_DIP:DIP-14_W7.62mm_LongPads, symbol custom:MCP6004
- added U?: SCD7805BTG, Package_TO_SOT_THT:TO-220-3_Horizontal_TabDown, symbol custom:SCD7805BTG
Connections:
- net labels added: +5V, 555_OUT
- net labels removed: DISCHARGE, FREQ_VFO_OUT, INV_TRIANGLE, SAW_EN
- wire segments 71 -> 84
Other:
- note added: "AMP"
- note added: "DUTY"
- note added: "FREQ"
- note added: "OFFSET"
- note removed: "ADD AMP/ATTEN + OFFSET STAGE"
- note removed: "MAKE SURE CLOCKWISE = INCREASE FREQ"
- note removed: "UPDATE SYMBOL"
- moved on the sheet: C?, R?, U?
