File: synth/synth.sch (KiCad schematic (older format))
At the start: 0 parts

Commit message: automated commit
Changed lines of the file:
@@
 $Descr A4 11693 8268
 encoding utf-8
-Sheet 1 4
+Sheet 1 5
 Title ""
 Date ""
@@
 $EndBitmap
 $Sheet
-S 1150 1025 1050 750
+S 2350 1050 1050 750
 U 5E4A00E6
-F0 "SWEEP_VFO" 50
-F1 "SWEEP_VFO.sch" 50
+F0 "FREQ_VFO" 50
+F1 "FREQ_VFO.sch" 50
 $EndSheet
 $Sheet
-S 2350 1025 1050 750
+S 3550 1050 1050 750
 U 5E4A00FF
-F0 "MODULATION_VFO." 50
-F1 "MODULATION_VFO.sch" 50
+F0 "AMP_VFO." 50
+F1 "AMP_VFO.sch" 50
 $EndSheet
 $Sheet
-S 3550 1025 1050 750
+S 4750 1050 1050 750
 U 5E4A013A
 F0 "MAIN_VFO" 50
 F1 "MAIN_VFO.sch" 50
 $EndSheet
+$Sheet
+S 1150 1050 1050 750
+U 5E69BAF5
+F0 "POWER" 50
+F1 "POWER.sch" 50
+$EndSheet
 $EndSCHEMATC
