File: synth/POWER.sch (KiCad schematic (older format))
At the start: 6 parts

Commit message: automated commit
Parts:
- added TP? (x2): PTH_1_mm, TestPoint:TestPoint_THTPad_D2.0mm_Drill1.0mm, symbol custom:PTH_1_mm
Connections:
- net GND: now also TP?.1, TP?.1
Changed lines of the file:
@@
 L power:GND #PWR?
 U 1 1 5E69BCFF
-P 6400 4400
+P 6400 4650
 AR Path="/5E69BCFF" Ref="#PWR?"  Part="1"
 AR Path="/5E4A00E6/5E69BCFF" Ref="#PWR?"  Part="1"
 AR Path="/5E69BAF5/5E69BCFF" Ref="#PWR?"  Part="1"
-F 0 "#PWR?" H 6400 4150 50  0001 C CNN
-F 1 "GND" H 6405 4227 50  0000 C CNN
-F 2 "" H 6400 4400 50  0001 C CNN
-F 3 "" H 6400 4400 50  0001 C CNN
-	1    6400 4400
+F 0 "#PWR?" H 6400 4400 50  0001 C CNN
+F 1 "GND" H 6405 4477 50  0000 C CNN
+F 2 "" H 6400 4650 50  0001 C CNN
+F 3 "" H 6400 4650 50  0001 C CNN
+	1    6400 4650
 	1    0    0    -1
 $EndComp
 Wire Wire Line
-	6400 4400 6400 4300
+	6400 4650 6400 4400
 Wire Wire Line
 	6400 3800 7000 3800
@@
 L power:GND #PWR?
 U 1 1 5E69BD28
-P 4250 4200
+P 4250 4500
 AR Path="/5E69BD28" Ref="#PWR?"  Part="1"
 AR Path="/5E4A00E6/5E69BD28" Ref="#PWR?"  Part="1"
 AR Path="/5E69BAF5/5E69BD28" Ref="#PWR?"  Part="1"
-F 0 "#PWR?" H 4250 3950 50  0001 C CNN
-F 1 "GND" H 4255 4027 50  0000 C CNN
-F 2 "" H 4250 4200 50  0001 C CNN
-F 3 "" H 4250 4200 50  0001 C CNN
-	1    4250 4200
+F 0 "#PWR?" H 4250 4250 50  0001 C CNN
+F 1 "GND" H 4255 4327 50  0000 C CNN
+F 2 "" H 4250 4500 50  0001 C CNN
+F 3 "" H 4250 4500 50  0001 C CNN
+	1    4250 4500
 	1    0    0    -1
 $EndComp
 Wire Wire Line
-	4250 4200 4250 4100
+	4250 4500 4250 4300
 $Comp
 L power:+5V #PWR?
@@
 	3550 3750 3700 3750
 Connection ~ 3700 3750
+$Comp
+L custom:PTH_1_mm TP?
+U 1 1 5E506E5B
+P 4550 4300
+F 0 "TP?" H 4500 4150 50  0000 L BNN
+F 1 "PTH_1_mm" H 4400 4050 50  0000 L BNN
+F 2 "TestPoint:TestPoint_THTPad_D2.0mm_Drill1.0mm" H 4350 4050 50  0001 L BNN
+F 3 "" H 4550 4400 50  0001 L BNN
+	1    4550 4300
+	1    0    0    -1
+$EndComp
+Wire Wire Line
+	4400 4300 4250 4300
+Connection ~ 4250 4300
+Wire Wire Line
+	4250 4300 4250 4100
+$Comp
+L custom:PTH_1_mm TP?
+U 1 1 5E507589
+P 6700 4400
+F 0 "TP?" H 6650 4250 50  0000 L BNN
+F 1 "PTH_1_mm" H 6550 4150 50  0000 L BNN
+F 2 "TestPoint:TestPoint_THTPad_D2.0mm_Drill1.0mm" H 6500 4150 50  0001 L BNN
+F 3 "" H 6700 4500 50  0001 L BNN
+	1    6700 4400
+	1    0    0    -1
+$EndComp
+Wire Wire Line
+	6550 4400 6400 4400
+Connection ~ 6400 4400
+Wire Wire Line
+	6400 4400 6400 4300
 $EndSCHEMATC
