File: synth/POWER.sch (KiCad schematic (older format))
At the start: 8 parts

Commit message: automated commit
Parts:
- removed TP? (x5): PTH_1_mm, TestPoint:TestPoint_THTPad_D2.0mm_Drill1.0mm, symbol custom:PTH_1_mm
- added C?: NP, symbol Device:CP1
- added JP?: SolderJumper_2_Open, symbol Jumper:SolderJumper_2_Open
- added TP? (x4): PTH_1_mm, TestPoint:TestPoint_THTPad_D2.0mm_Drill1.0mm, symbol custom:PTH_1_mm
Connections:
- net +5V: now also JP?.2 (B), TP?.1
- net GND: now also C?.2, TP?.1
- net HI_Z_REF: now also C?.1, TP?.1
- net VDD_BAT: now also JP?.1 (A), TP?.1
Other:
- note added: "NEED TO ADD BATTERY HOLDER"
- note added: "SILKSCREEN:\nWARNING: DO NOT CONNECT\nUNLESS BOARD IS CONVERTED\nTO OPERATE AT HIGHER VOLTAGES.\nALTERNATIVE PARTS REQUIRED."
Changed lines of the file:
@@
 L power:GND #PWR?
 U 1 1 5E69BCFF
-P 6400 4650
+P 6400 4500
 AR Path="/5E69BCFF" Ref="#PWR?"  Part="1"
 AR Path="/5E4A00E6/5E69BCFF" Ref="#PWR?"  Part="1"
 AR Path="/5E69BAF5/5E69BCFF" Ref="#PWR?"  Part="1"
-F 0 "#PWR?" H 6400 4400 50  0001 C CNN
-F 1 "GND" H 6405 4477 50  0000 C CNN
-F 2 "" H 6400 4650 50  0001 C CNN
-F 3 "" H 6400 4650 50  0001 C CNN
-	1    6400 4650
-	1    0    0    -1
-$EndComp
-Wire Wire Line
-	6400 4650 6400 4400
-Wire Wire Line
-	6400 3800 7000 3800
+F 0 "#PWR?" H 6400 4250 50  0001 C CNN
+F 1 "GND" H 6405 4327 50  0000 C CNN
+F 2 "" H 6400 4500 50  0001 C CNN
+F 3 "" H 6400 4500 50  0001 C CNN
+	1    6400 4500
+	1    0    0    -1
+$EndComp
+Wire Wire Line
+	6400 3800 6750 3800
 Connection ~ 6400 3800
 Wire Wire Line
@@
 	1    0    0    -1
 $EndComp
-Text GLabel 7400 3800 2    50   Output ~ 0
+Text GLabel 7300 3800 2    50   Output ~ 0
 HI_Z_REF
-$Comp
-L custom:PTH_1_mm TP?
-U 1 1 5E6F5FAC
-P 7000 3500
-F 0 "TP?" V 7250 3450 50  0000 L BNN
-F 1 "PTH_1_mm" V 7150 3300 50  0000 L BNN
-F 2 "TestPoint:TestPoint_THTPad_D2.0mm_Drill1.0mm" H 6800 3250 50  0001 L BNN
-F 3 "" H 7000 3600 50  0001 L BNN
-	1    7000 3500
+Wire Wire Line
+	6750 3750 6750 3800
+Connection ~ 6750 3800
+Wire Wire Line
+	6750 3800 7150 3800
+Wire Wire Line
+	3650 3750 3700 3750
+Connection ~ 3700 3750
+Wire Wire Line
+	4300 4300 4250 4300
+Connection ~ 4250 4300
+Wire Wire Line
+	4250 4300 4250 4100
+$Comp
+L custom:PTH_1_mm TP?
+U 1 1 5E61F9DD
+P 6750 3600
+AR Path="/5E4A00E6/5E61F9DD" Ref="TP?"  Part="1"
+AR Path="/5E69BAF5/5E61F9DD" Ref="TP?"  Part="1"
+F 0 "TP?" V 6850 3550 50  0000 L BNN
+F 1 "PTH_1_mm" V 6900 3400 50  0001 L BNN
+F 2 "TestPoint:TestPoint_THTPad_D2.0mm_Drill1.0mm" H 6550 3350 50  0001 L BNN
+F 3 "" H 6750 3700 50  0001 L BNN
+	1    6750 3600
 	0    -1   -1   0
 $EndComp
-Wire Wire Line
-	7000 3650 7000 3800
-Connection ~ 7000 3800
-Wire Wire Line
-	7000 3800 7400 3800
-$Comp
-L custom:PTH_1_mm TP?
-U 1 1 5E6F62FB
-P 5150 3750
-F 0 "TP?" H 5100 3600 50  0000 L BNN
-F 1 "PTH_1_mm" H 5000 3500 50  0000 L BNN
-F 2 "TestPoint:TestPoint_THTPad_D2.0mm_Drill1.0mm" H 4950 3500 50  0001 L BNN
-F 3 "" H 5150 3850 50  0001 L BNN
-	1    5150 3750
-	1    0    0    -1
-$EndComp
-Wire Wire Line
-	5000 3750 4850 3750
+$Comp
+L custom:PTH_1_mm TP?
+U 1 1 5E61FC80
+P 5050 3750
+AR Path="/5E4A00E6/5E61FC80" Ref="TP?"  Part="1"
+AR Path="/5E69BAF5/5E61FC80" Ref="TP?"  Part="1"
+F 0 "TP?" H 5100 3750 50  0000 L BNN
+F 1 "PTH_1_mm" V 5200 3550 50  0001 L BNN
+F 2 "TestPoint:TestPoint_THTPad_D2.0mm_Drill1.0mm" H 4850 3500 50  0001 L BNN
+F 3 "" H 5050 3850 50  0001 L BNN
+	1    5050 3750
+	1    0    0    -1
+$EndComp
+Wire Wire Line
+	4900 3750 4850 3750
 Connection ~ 4850 3750
 $Comp
 L custom:PTH_1_mm TP?
-U 1 1 5E6F68D1
-P 3400 3750
-F 0 "TP?" H 3350 3850 50  0000 L BNN
-F 1 "PTH_1_mm" H 3250 3950 50  0000 L BNN
-F 2 "TestPoint:TestPoint_THTPad_D2.0mm_Drill1.0mm" H 3200 3500 50  0001 L BNN
-F 3 "" H 3400 3850 50  0001 L BNN
-	1    3400 3750
+U 1 1 5E6200E9
+P 3500 3750
+AR Path="/5E4A00E6/5E6200E9" Ref="TP?"  Part="1"
+AR Path="/5E69BAF5/5E6200E9" Ref="TP?"  Part="1"
+F 0 "TP?" H 3550 3750 50  0000 L BNN
+F 1 "PTH_1_mm" V 3650 3550 50  0001 L BNN
+F 2 "TestPoint:TestPoint_THTPad_D2.0mm_Drill1.0mm" H 3300 3500 50  0001 L BNN
+F 3 "" H 3500 3850 50  0001 L BNN
+	1    3500 3750
 	-1   0    0    1
 $EndComp
-Wire Wire Line
-	3550 3750 3700 3750
-Connection ~ 3700 3750
-$Comp
-L custom:PTH_1_mm TP?
-U 1 1 5E506E5B
-P 4550 4300
-F 0 "TP?" H 4500 4150 50  0000 L BNN
-F 1 "PTH_1_mm" H 4400 4050 50  0000 L BNN
-F 2 "TestPoint:TestPoint_THTPad_D2.0mm_Drill1.0mm" H 4350 4050 50  0001 L BNN
-F 3 "" H 4550 4400 50  0001 L BNN
-	1    4550 4300
-	1    0    0    -1
-$EndComp
-Wire Wire Line
-	4400 4300 4250 4300
-Connection ~ 4250 4300
-Wire Wire Line
-	4250 4300 4250 4100
-$Comp
-L custom:PTH_1_mm TP?
-U 1 1 5E507589
-P 6700 4400
-F 0 "TP?" H 6650 4250 50  0000 L BNN
-F 1 "PTH_1_mm" H 6550 4150 50  0000 L BNN
-F 2 "TestPoint:TestPoint_THTPad_D2.0mm_Drill1.0mm" H 6500 4150 50  0001 L BNN
-F 3 "" H 6700 4500 50  0001 L BNN
-	1    6700 4400
-	1    0    0    -1
-$EndComp
-Wire Wire Line
-	6550 4400 6400 4400
-Connection ~ 6400 4400
-Wire Wire Line
-	6400 4400 6400 4300
+$Comp
+L custom:PTH_1_mm TP?
+U 1 1 5E62014F
+P 4450 4300
+AR Path="/5E4A00E6/5E62014F" Ref="TP?"  Part="1"
+AR Path="/5E69BAF5/5E62014F" Ref="TP?"  Part="1"
+F 0 "TP?" H 4500 4300 50  0000 L BNN
+F 1 "PTH_1_mm" V 4600 4100 50  0001 L BNN
+F 2 "TestPoint:TestPoint_THTPad_D2.0mm_Drill1.0mm" H 4250 4050 50  0001 L BNN
+F 3 "" H 4450 4400 50  0001 L BNN
+	1    4450 4300
+	1    0    0    -1
+$EndComp
+$Comp
+L Jumper:SolderJumper_2_Open JP?
+U 1 1 5E7C023F
+P 5250 5450
+F 0 "JP?" H 5250 5530 50  0000 C CNN
+F 1 "SolderJumper_2_Open" H 5250 5350 50  0001 C CNN
+F 2 "" H 5250 5450 50  0001 C CNN
+F 3 "~" H 5250 5450 50  0001 C CNN
+	1    5250 5450
+	1    0    0    -1
+$EndComp
+$Comp
+L custom:VDD_BAT #PWR?
+U 1 1 5E7C0A6B
+P 4900 5250
+AR Path="/5E4A00E6/5E7C0A6B" Ref="#PWR?"  Part="1"
+AR Path="/5E7C0A6B" Ref="#PWR?"  Part="1"
+AR Path="/5E69BAF5/5E7C0A6B" Ref="#PWR?"  Part="1"
+F 0 "#PWR?" H 5100 5300 50  0001 C CNN
+F 1 "VDD_BAT" H 4750 5400 50  0000 L BNN
+F 2 "" H 4900 5250 50  0001 C CNN
+F 3 "" H 4900 5250 50  0001 C CNN
+	1    4900 5250
+	1    0    0    -1
+$EndComp
+$Comp
+L power:+5V #PWR?
+U 1 1 5E7C0A88
+P 5600 5250
+AR Path="/5E4A00E6/5E7C0A88" Ref="#PWR?"  Part="1"
+AR Path="/5E7C0A88" Ref="#PWR?"  Part="1"
+AR Path="/5E69BAF5/5E7C0A88" Ref="#PWR?"  Part="1"
+F 0 "#PWR?" H 5600 5100 50  0001 C CNN
+F 1 "+5V" H 5600 5390 50  0000 C CNN
+F 2 "" H 5600 5250 50  0001 C CNN
+F 3 "" H 5600 5250 50  0001 C CNN
+	1    5600 5250
+	1    0    0    -1
+$EndComp
+Wire Wire Line
+	4900 5250 4900 5450
+Wire Wire Line
+	4900 5450 5100 5450
+Wire Wire Line
+	5400 5450 5600 5450
+Wire Wire Line
+	5600 5450 5600 5250
+Text Notes 4700 5950 0    50   ~ 0
+SILKSCREEN:\nWARNING: DO NOT CONNECT\nUNLESS BOARD IS CONVERTED\nTO OPERATE AT HIGHER VOLTAGES.\nALTERNATIVE PARTS REQUIRED.
+$Comp
+L Device:CP1 C?
+U 1 1 5E7C9010
+P 7150 4150
+F 0 "C?" H 7175 4250 50  0000 L CNN
+F 1 "NP" H 7175 4050 50  0000 L CNN
+F 2 "" H 7150 4150 50  0001 C CNN
+F 3 "~" H 7150 4150 50  0001 C CNN
+	1    7150 4150
+	1    0    0    -1
+$EndComp
+Wire Wire Line
+	7150 4000 7150 3800
+Connection ~ 7150 3800
+Wire Wire Line
+	7150 3800 7300 3800
+$Comp
+L power:GND #PWR?
+U 1 1 5E7C9456
+P 7150 4500
+AR Path="/5E7C9456" Ref="#PWR?"  Part="1"
+AR Path="/5E4A00E6/5E7C9456" Ref="#PWR?"  Part="1"
+AR Path="/5E69BAF5/5E7C9456" Ref="#PWR?"  Part="1"
+F 0 "#PWR?" H 7150 4250 50  0001 C CNN
+F 1 "GND" H 7155 4327 50  0000 C CNN
+F 2 "" H 7150 4500 50  0001 C CNN
+F 3 "" H 7150 4500 50  0001 C CNN
+	1    7150 4500
+	1    0    0    -1
+$EndComp
+Wire Wire Line
+	7150 4500 7150 4300
+Wire Wire Line
+	6400 4300 6400 4500
+Text Notes 5000 2400 0    50   ~ 0
+NEED TO ADD BATTERY HOLDER
 $EndSCHEMATC
