File: synth/AMP_VFO.sch (KiCad schematic (older format))
At the start: 0 parts

Commit message: automated commit
Parts:
- added C?: 10uF, symbol Device:CP1
- added C? (x2): 1uF, symbol Device:CP1
- added D?: D_Schottky_Small_ALT, symbol Device:D_Schottky_Small_ALT
- added JP? (x2): SolderJumper_2_Bridged, symbol Jumper:SolderJumper_2_Bridged
- added Q?: BC549BTA, symbol Device:Q_NPN_CBE
- added Q?: BC556BTA, symbol Device:Q_PNP_CBE
- added R?: NP_100, symbol Device:R
- added R? (x3): 10k, symbol Device:R
- added R? (x4): 3k3, symbol Device:R
- added R?: 5k, symbol Device:R
- added R?: NP_10k, symbol Device:R
- added RV? (x4): 10k, symbol Device:R_POT
- added SW?: SW_SPDT, symbol Switch:SW_SPDT
- added TP? (x10): PTH_1_mm, TestPoint:TestPoint_THTPad_D2.0mm_Drill1.0mm, symbol custom:PTH_1_mm
- added U?: SE555P, symbol custom:SE555P
- added U? (x5): MCP6004, Package_DIP:DIP-14_W7.62mm_LongPads, symbol custom:MCP6004
Connections:
- new net: R?.1, R?.2, R?.2, U?.3 (OUT)
- new net: C?.2, D?.2 (A), JP?.1 (A), R?.2, TP?.1, U?.6 (-)
- new net: JP?.2 (B), R?.1, RV?.2, TP?.1
- new net: R?.2, RV?.1, U?.2 (-)
- new net: Q?.3 (E), Q?.3 (E), RV?.2, TP?.1, U?.1
- new net: R?.1, R?.2, R?.2, TP?.1, U?.10 (+)
- new net: JP?.2 (B), R?.1, R?.2, SW?.3 (C), TP?.1, U?.8
- new net: JP?.1 (A), R?.2, TP?.1, U?.9 (-)
- new net: RV?.2, TP?.1, U?.12 (+)
- new net: R?.2, RV?.1, U?.13 (-)
- new net: Q?.1 (C), RV?.1
- new net: Q?.2 (B), R?.1 (x2)
- new net: Q?.1 (C), RV?.3
- new net: R?.1, SW?.2 (B)
- new net +5V: C?.1, C?.1, R?.1, RV?.3, U?.4 (V+), U?.4 (~R), U?.8 (VCC)
- new net AMP_VFO: RV?.2, TP?.1, U?.14
- new net DISCHARGE: R?.2, U?.7 (DISCH)
- new net GND: C?.2, C?.2, R?.1, R?.1, RV?.1, TP?.1, U?.1 (GND), U?.11 (V-)
- new net HI_Z_REF: U?.3 (+), U?.5 (+)
- new net TRIANGLE: C?.1, D?.1 (K), SW?.1 (A), TP?.1, U?.2 (TRIG), U?.6 (THR), U?.7
- no-connect marks 0 -> 3
Other:
- note added: "AMP"
- note added: "DUTY"
- note added: "FREQ"
- note added: "LINEAR"
- note added: "LOGARITHMIC"
- note added: "OFFSET"
- note added: "SQUARE"
- note added: "TR/SQ"
- note added: "TURN INTO INV LOG CONFIGURATION?"
