File: synth/MAIN_VFO.sch (KiCad schematic (older format))
At the start: 4 parts

Commit message: automated commit
Parts:
- removed U?: SE555P, symbol custom:SE555P
- removed U? (x3): LM358P, Package_DIP:DIP-8_W7.62mm, symbol custom:LM358P
Connections:
- net labels removed: GND, VDD_BAT
- wire segments 4 -> 0
Changed lines of the file:
@@
 EELAYER 26 0
 EELAYER END
-$Descr A4 11693 8268
+$Descr USLetter 11000 8500
 encoding utf-8
-Sheet 4 4
+Sheet 4 5
 Title ""
 Date ""
@@
 Comment4 ""
 $EndDescr
-$Comp
-L power:GND #PWR?
-U 1 1 5E4A0672
-P 8075 4525
-F 0 "#PWR?" H 8075 4275 50  0001 C CNN
-F 1 "GND" H 8080 4352 50  0000 C CNN
-F 2 "" H 8075 4525 50  0001 C CNN
-F 3 "" H 8075 4525 50  0001 C CNN
-	1    8075 4525
-	1    0    0    -1
-$EndComp
-$Comp
-L custom:VDD_BAT #PWR?
-U 1 1 5E4A0678
-P 7075 3625
-F 0 "#PWR?" H 7275 3675 50  0001 C CNN
-F 1 "VDD_BAT" H 7080 3798 50  0000 C CNN
-F 2 "" H 7075 3625 50  0001 C CNN
-F 3 "" H 7075 3625 50  0001 C CNN
-	1    7075 3625
-	1    0    0    -1
-$EndComp
-Wire Wire Line
-	7075 3625 7075 3750
-Wire Wire Line
-	7075 3750 7175 3750
-Wire Wire Line
-	8075 4525 8075 4350
-Wire Wire Line
-	8075 4350 7975 4350
-$Comp
-L custom:SE555P U?
-U 1 1 5E4A0682
-P 7575 4250
-F 0 "U?" H 7575 5017 50  0000 C CNN
-F 1 "SE555P" H 7575 4926 50  0000 C CNN
-F 2 "" H 7575 4250 50  0001 C CNN
-F 3 "http://www.ti.com/lit/ds/symlink/lm555.pdf" H 7575 4250 50  0001 C CNN
-	1    7575 4250
-	1    0    0    -1
-$EndComp
-$Comp
-L custom:LM358P U?
-U 1 1 5E4A0689
-P 4200 2775
-F 0 "U?" H 4200 3142 50  0000 C CNN
-F 1 "LM358P" H 4200 3051 50  0000 C CNN
-F 2 "Package_DIP:DIP-8_W7.62mm" H 4200 2225 50  0001 C CNN
-F 3 "~/dj/datasheets/LM358P.pdf" H 4200 2325 50  0001 C CNN
-	1    4200 2775
-	1    0    0    -1
-$EndComp
-$Comp
-L custom:LM358P U?
-U 2 1 5E4A0690
-P 4100 3475
-F 0 "U?" H 4100 3842 50  0000 C CNN
-F 1 "LM358P" H 4100 3751 50  0000 C CNN
-F 2 "Package_DIP:DIP-8_W7.62mm" H 4100 2925 50  0001 C CNN
-F 3 "~/dj/datasheets/LM358P.pdf" H 4100 3025 50  0001 C CNN
-	2    4100 3475
-	1    0    0    -1
-$EndComp
-$Comp
-L custom:LM358P U?
-U 3 1 5E4A0697
-P 3750 4050
-F 0 "U?" H 3980 4096 50  0000 L CNN
-F 1 "LM358P" H 3980 4005 50  0000 L CNN
-F 2 "Package_DIP:DIP-8_W7.62mm" H 3750 3500 50  0001 C CNN
-F 3 "~/dj/datasheets/LM358P.pdf" H 3750 3600 50  0001 C CNN
-	3    3750 4050
-	1    0    0    -1
-$EndComp
 $EndSCHEMATC

Commit message: automated commit
Parts:
- added C?: 10uF, symbol Device:CP1
- added C? (x2): 1uF, symbol Device:CP1
- added D?: D_Schottky_Small_ALT, symbol Device:D_Schottky_Small_ALT
- added JP? (x2): SolderJumper_2_Bridged, symbol Jumper:SolderJumper_2_Bridged
- added Q?: BC549BTA, symbol Device:Q_NPN_CBE
- added Q?: BC556BTA, symbol Device:Q_PNP_CBE
- added R?: NP_100, symbol Device:R
- added R? (x4): 10k, symbol Device:R
- added R? (x4): 3k3, symbol Device:R
- added R?: 5k, symbol Device:R
- added R?: NP_10k, symbol Device:R
- added RV? (x3): 10k, symbol Device:R_POT
- added SW?: SW_SPDT, symbol Switch:SW_SPDT
- added TP? (x10): PTH_1_mm, TestPoint:TestPoint_THTPad_D2.0mm_Drill1.0mm, symbol custom:PTH_1_mm
- added U?: SE555P, symbol custom:SE555P
- added U? (x5): MCP6004, Package_DIP:DIP-14_W7.62mm_LongPads, symbol custom:MCP6004
Connections:
- new net: R?.2, R?.2, U?.3 (OUT)
- new net: C?.2, D?.2 (A), JP?.1 (A), R?.2, TP?.1, U?.6 (-)
- new net: JP?.2 (B), R?.1, RV?.2, TP?.1
- new net: R?.1, R?.2, U?.2 (-)
- new net: Q?.3 (E), R?.2, TP?.1, U?.1
- new net: R?.1, R?.2, R?.2, TP?.1, U?.10 (+)
- new net: JP?.2 (B), R?.1, R?.2, SW?.3 (C), TP?.1, U?.8
- new net: JP?.1 (A), R?.2, TP?.1, U?.9 (-)
- new net: RV?.2, TP?.1, U?.12 (+)
- new net: R?.2, RV?.1, U?.13 (-)
- new net: Q?.1 (C), RV?.1
- new net: Q?.2 (B), R?.1 (x2)
- new net: Q?.1 (C), RV?.3
- new net: R?.1, SW?.2 (B)
- new net +5V: C?.1, C?.1, R?.1, RV?.3, U?.4 (V+), U?.4 (~R), U?.8 (VCC)
- new net DISCHARGE: R?.2, U?.7 (DISCH)
- new net FREQ_VFO: Q?.3 (E), R?.1, RV?.2, TP?.1, U?.14
- new net GND: C?.2, C?.2, R?.1, R?.1, RV?.1, TP?.1, U?.1 (GND), U?.11 (V-)
- new net HI_Z_REF: U?.3 (+), U?.5 (+)
- new net TRIANGLE: C?.1, D?.1 (K), SW?.1 (A), TP?.1, U?.2 (TRIG), U?.6 (THR), U?.7
- no-connect marks 0 -> 2
Other:
- note added: "AMP"
- note added: "DUTY"
- note added: "LINEAR"
- note added: "LOGARITHMIC"
- note added: "OFFSET"
- note added: "SQUARE"
- note added: "TR/SQ"
