File: synth/MAIN_VFO.sch (KiCad schematic (older format))
At the start: 39 parts

Commit message: automated commit
Parts:
- C?: value 10uF -> 100nF
Changed lines of the file:
@@
 AR Path="/5E4A013A/5E527227" Ref="C?"  Part="1"
 F 0 "C?" V 6350 1600 50  0000 C CNN
-F 1 "10uF" V 6350 1950 50  0000 C CNN
+F 1 "100nF" V 6350 2000 50  0000 C CNN
 F 2 "" H 6300 1800 50  0001 C CNN
 F 3 "~" H 6300 1800 50  0001 C CNN
