File: synth/FREQ_VFO.sch (KiCad schematic (older format))
At the start: 27 parts

Commit message: automated commit
Parts:
- removed TP?: PTH_1_mm, TestPoint:TestPoint_THTPad_D2.0mm_Drill1.0mm, symbol custom:PTH_1_mm
- added NP_C? (x2): 1uF, symbol Device:CP1
- added TP? (x5): PTH_1_mm, TestPoint:TestPoint_THTPad_D2.0mm_Drill1.0mm, symbol custom:PTH_1_mm
Connections:
- net +5V: now also NP_C?.1, NP_C?.1
- net FREQ_VFO: now also TP?.1
- net GND: now also NP_C?.2, NP_C?.2, TP?.1
- net at C?.2, R?.2, U?.6 (-): now also TP?.1
- net at R?.1, RV?.2: now also TP?.1
- net at R?.1, R?.2, U?.9 (-): now also TP?.1
Other:
- moved on the sheet: Q?, R?, RV?, TP?, U?A, U?E

Commit message: automated commit
Parts:
- removed R? (x3): 10k, symbol Device:R
- removed R?: 3k3, symbol Device:R
- removed TP? (x8): PTH_1_mm, TestPoint:TestPoint_THTPad_D2.0mm_Drill1.0mm, symbol custom:PTH_1_mm
- added D?: D_Schottky_Small_ALT, symbol Device:D_Schottky_Small_ALT
- added JP? (x2): SolderJumper_2_Bridged, symbol Jumper:SolderJumper_2_Bridged
- added R?: 5k, symbol Device:R
- added R? (x2): 10k, symbol Device:R
- added R? (x3): 3k3, symbol Device:R
- added R?: NP_10k, symbol Device:R
- added TP? (x8): PTH_1_mm, TestPoint:TestPoint_THTPad_D2.0mm_Drill1.0mm, symbol custom:PTH_1_mm
- C? (x2): renamed from NP_C?; NP (none) -> NP
- R?: value 680 -> NP_100
Connections:
- net +5V: now also RV?.3, R?.1; no longer RV?.1
- net FREQ_VFO: now also TP?.1
- net GND: now also RV?.1, R?.1, R?.1; no longer RV?.3
- net HI_Z_REF: no longer U?.10 (+)
- net TRIANGLE: now also D?.1 (K)
- net DISCHARGE: now reaches U?.7 (DISCH)
- net DISCHARGE: now also R?.2
- net at C?.2, R?.2, U?.6 (-): now also D?.2 (A), JP?.1 (A), TP?.1
- net at R?.1, RV?.2: now also JP?.2 (B), TP?.1
- net at R?.2, U?.2 (-): now also RV?.1; no longer RV?.3
- net at Q?.3 (E), Q?.3 (E), RV?.2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: now also TP?.1
- net at Q?.2 (B): now also R?.1 (x2)
- net at U?.9 (-): now also JP?.1 (A), R?.2, TP?.1
- net at RV?.2, U?.12 (+): now also TP?.1
- net at R?.2, U?.13 (-): now also RV?.1; no longer RV?.3
- net at Q?.1 (C): now also RV?.1; no longer RV?.3
- net at Q?.1 (C): now also RV?.3; no longer RV?.1
- net 555_OUT: no longer names the net of R?.1, U?.3 (OUT)
- net 555_OUT: now also R?.2, R?.2
- net SQUARE: no longer names the net of SW?.3 (C), U?.8
- net SQUARE: now also JP?.2 (B), R?.1, R?.2, TP?.1
- new net: R?.1, R?.2, R?.2, TP?.1, U?.10 (+)
- no-connect marks 4 -> 3
Other:
- note added: "LINEAR"
- note added: "LOGARITHMIC"
- note added: "SQUARE"
- note added: "TR/SQ"
- moved on the sheet: C?, Q?, R?, RV?, SW?, TP?, U?, U?A, U?B, U?C, U?D, U?E

Commit message: automated commit
Parts:
- removed JP?: SolderJumper_2_Bridged, symbol Jumper:SolderJumper_2_Bridged
- removed R? (x2): 10k, symbol Device:R
- removed R?: NP_10k, symbol Device:R
- removed TP? (x3): PTH_1_mm, TestPoint:TestPoint_THTPad_D2.0mm_Drill1.0mm, symbol custom:PTH_1_mm
- removed U?: MCP6004, Package_DIP:DIP-14_W7.62mm_LongPads, symbol custom:MCP6004
- added R? (x2): 3k3, symbol Device:R
- added RV?: 10k, symbol Device:R_POT
Connections:
- wire segments 112 -> 102
Other:
- note added: "OFFSET STAGE\n"
- moved on the sheet: C?, R?, RV?, SW?, TP?, U?D, U?E

Commit message: automated commit
Parts:
- removed R? (x2): 3k3, symbol Device:R
- added R?: 10k, symbol Device:R
- RV?: value 10k -> 15k
Connections:
- wire segments 102 -> 101
- no-connect marks 3 -> 4
Other:
- moved on the sheet: RV?, U?D
Changed lines of the file:
@@
 L custom:MCP6004 U?
 U 4 1 5E50F5B4
-P 6350 5000
-F 0 "U?" H 6150 4750 50  0000 L CNN
-F 1 "MCP6004" H 6150 5250 50  0000 L CNN
-F 2 "Package_DIP:DIP-14_W7.62mm_LongPads" H 6350 4400 50  0001 C CNN
-F 3 "~/home/dj/datasheets/MCP6004.pdf" H 6350 4550 50  0001 C CNN
-	4    6350 5000
+P 6100 5000
+F 0 "U?" H 5900 4750 50  0000 L CNN
+F 1 "MCP6004" H 5900 5250 50  0000 L CNN
+F 2 "Package_DIP:DIP-14_W7.62mm_LongPads" H 6100 4400 50  0001 C CNN
+F 3 "~/home/dj/datasheets/MCP6004.pdf" H 6100 4550 50  0001 C CNN
+	4    6100 5000
 	1    0    0    1
 $EndComp
@@
 Wire Wire Line
 	1900 2350 2000 2350
-Text Notes 12150 4600 0    79   ~ 16
+Text Notes 5650 4350 0    79   ~ 16
 AMP
 Text GLabel 2450 2550 0    50   Input ~ 0
@@
 	3600 4800 3600 5000
 Wire Wire Line
-	5950 5100 6050 5100
+	6550 5000 6400 5000
+Wire Wire Line
+	5550 4900 5800 4900
+$Comp
+L Device:R_POT RV?
+U 1 1 5E6409C9
+P 5550 4500
+F 0 "RV?" V 5450 4600 50  0000 R CNN
+F 1 "15k" V 5550 4550 39  0000 R CNN
+F 2 "" H 5550 4500 50  0001 C CNN
+F 3 "~" H 5550 4500 50  0001 C CNN
+	1    5550 4500
+	1    0    0    1
+$EndComp
+Wire Wire Line
+	5550 4650 5550 4900
+Wire Wire Line
+	5700 4500 6550 4500
+Wire Wire Line
+	6550 4500 6550 5000
+Wire Wire Line
+	4900 4900 5000 4900
+Connection ~ 5550 4900
+Text Notes 7500 4900 0    50   ~ 0
+OFFSET STAGE\n
 $Comp
 L Device:R R?
-U 1 1 5E5C4319
+U 1 1 5E52C38C
 P 5150 4900
 F 0 "R?" V 5225 4900 50  0000 L CNN
-F 1 "3k3" V 5150 4850 39  0000 L CNN
+F 1 "10k" V 5150 4850 39  0000 L CNN
 F 2 "" V 5080 4900 50  0001 C CNN
 F 3 "~" H 5150 4900 50  0001 C CNN
@@
 $EndComp
 Wire Wire Line
-	6800 5000 6650 5000
-Wire Wire Line
-	5800 4900 6050 4900
-$Comp
-L power:GND #PWR?
-U 1 1 5E60F429
-P 5950 5350
-AR Path="/5E60F429" Ref="#PWR?"  Part="1"
-AR Path="/5E4A00E6/5E60F429" Ref="#PWR?"  Part="1"
-F 0 "#PWR?" H 5950 5100 50  0001 C CNN
-F 1 "GND" H 5955 5177 50  0000 C CNN
-F 2 "" H 5950 5350 50  0001 C CNN
-F 3 "" H 5950 5350 50  0001 C CNN
-	1    5950 5350
-	1    0    0    -1
-$EndComp
-Wire Wire Line
-	5950 5350 5950 5100
-$Comp
-L Device:R_POT RV?
-U 1 1 5E6409C9
-P 5800 4500
-F 0 "RV?" V 5700 4600 50  0000 R CNN
-F 1 "10k" V 5800 4550 39  0000 R CNN
-F 2 "" H 5800 4500 50  0001 C CNN
-F 3 "~" H 5800 4500 50  0001 C CNN
-	1    5800 4500
-	1    0    0    1
-$EndComp
-Wire Wire Line
-	5800 4650 5800 4900
-Wire Wire Line
-	5950 4500 6800 4500
-Wire Wire Line
-	6800 4500 6800 5000
-$Comp
-L Device:R R?
-U 1 1 5E64C497
-P 5550 4900
-F 0 "R?" V 5625 4900 50  0000 L CNN
-F 1 "3k3" V 5550 4850 39  0000 L CNN
-F 2 "" V 5480 4900 50  0001 C CNN
-F 3 "~" H 5550 4900 50  0001 C CNN
-	1    5550 4900
-	0    -1   -1   0
-$EndComp
-Wire Wire Line
-	4900 4900 5000 4900
-Wire Wire Line
-	5300 4900 5400 4900
-Wire Wire Line
-	5700 4900 5800 4900
-Connection ~ 5800 4900
-Text Notes 7500 4900 0    50   ~ 0
-OFFSET STAGE\n
+	5300 4900 5550 4900
+NoConn ~ 5550 4300
+Wire Wire Line
+	5550 4350 5550 4300
+Wire Wire Line
+	5600 5100 5800 5100
+Text GLabel 5600 5100 0    50   Input ~ 0
+HI_Z_REF
 $EndSCHEMATC

Commit message: automated commit
Parts:
- removed R?: 3k3, symbol Device:R
- removed RV? (x2): 10k, symbol Device:R_POT
- removed TP? (x2): PTH_1_mm, TestPoint:TestPoint_THTPad_D2.0mm_Drill1.0mm, symbol custom:PTH_1_mm
- added R? (x6): 10k, symbol Device:R
- added RV?: 10k, symbol Device:R_POT
- added U?: MCP6004, symbol Amplifier_Operational:MCP6004
- added U?: MCP6004, Package_DIP:DIP-14_W7.62mm_LongPads, symbol custom:MCP6004
- RV?: value 15k -> 7k5
Connections:
- net labels added: OFFSET
- wire segments 101 -> 112
- no-connect marks 4 -> 3
Other:
- note removed: "LOGARITHMIC"
- note removed: "OFFSET STAGE\n"
- moved on the sheet: C?, D?, JP?, Q?, R?, RV?, SW?, TP?, U?, U?A, U?B, U?D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

Commit message: automated commit
Parts:
- removed R?: 10k, symbol Device:R
- added C? (x4): NP, symbol Device:C
- RV?: value 7k5 -> 15k
Connections:
- net +5V: now also RV?.3
- net GND: now also C?.2, C?.2, C?.2, C?.2
- net at C?.2, D?.2 (A), JP?.1 (A)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: now also C?.1
- net at R?.2, RV?.1, U?.2 (-): now also C?.1
- net at R?.2, R?.2, U?.12 (+): now also C?.1
- net at R?.1, RV?.1, U?.9 (-): now also C?.1
Other:
- moved on the sheet: C?, D?, R?, RV?, TP?, U?, U?B, U?C, U?D
